Commit message: Site update 周日 2025/12/28 10:48:53.77

File: assets/robot_model/d1h/urdf/robot.urdf (robot description, URDF)
Before this commit: robot d1h_description, 13 links, 12 joints
Links:
- link FL_calf: geometry collision box size=0.24 0.04 0.05; visual mesh filename=../meshes/L_calf.STL
- link FL_foot: geometry collision cylinder length=0.04 radius=0.087; visual mesh filename=../meshes/L_foot.STL
- link FL_hip: geometry visual mesh filename=../meshes/L_hip.STL
- link FL_thigh: geometry collision box size=0.26 0.09 0.05; visual mesh filename=../meshes/L_thigh.STL
- link FR_calf: geometry collision box size=0.24 0.04 0.05; visual mesh filename=../meshes/R_calf.STL
- link FR_foot: geometry collision cylinder length=0.04 radius=0.087; visual mesh filename=../meshes/R_foot.STL
- link FR_hip: geometry visual mesh filename=../meshes/R_hip.STL
- link FR_thigh: geometry collision box size=0.26 0.09 0.05; visual mesh filename=../meshes/R_thigh.STL
- link F_base_link: geometry collision box size=0.275 0.15 0.175; collision box size=0.31 0.12 0.06
- link F_docking_link: geometry collision box size=0.0851 0.15 0.175; visual mesh filename=../meshes/docking_Link.STL
- link F_funtion_link: geometry collision box size=0.0495 0.15 0.175; visual mesh filename=../meshes/funtion_Link.STL

File: assets/robot_model/tita/urdf/robot.urdf (robot description, URDF)
Before this commit: robot tita, 15 links, 14 joints
Links:
- link base_link: geometry collision box size=0.47 0.3 0.19; visual mesh filename=../meshes/base_link.STL
- link left_leg_1: geometry visual mesh filename=../meshes/left_leg_1.STL
- link left_leg_2: geometry visual mesh filename=../meshes/left_leg_2.STL
- link left_leg_3: geometry collision box size=0.2 0.07 0.05; visual mesh filename=../meshes/left_leg_3.STL
- link left_leg_4: geometry collision cylinder length=0.034 radius=0.0925; visual mesh filename=../meshes/left_leg_4.STL
- link right_leg_1: geometry visual mesh filename=../meshes/right_leg_1.STL
- link right_leg_2: geometry visual mesh filename=../meshes/right_leg_2.STL
- link right_leg_3: geometry collision box size=0.2 0.07 0.05; visual mesh filename=../meshes/right_leg_3.STL
- link right_leg_4: geometry collision cylinder length=0.034 radius=0.0925; visual mesh filename=../meshes/right_leg_4.STL
