Commit message: 2026-03-10 20:59:56

File: assets/robot_model/duow/urdf/duow.urdf (robot description, URDF)
Before this commit: robot duow, 11 links, 10 joints
Joints:
- joint FL_hip_joint: limit lower=-0.36 upper=0.61 effort=36 velocity=42 -> lower=-0.61 upper=0.36 effort=36 velocity=42
- joint FR_hip_joint: limit lower=-0.61 upper=0.36 effort=36 velocity=42 -> lower=-0.36 upper=0.61 effort=36 velocity=42
